File: fezzesarecool-elec.kicad_pcb (KiCad board)
At the start: 2 copper layers, 65 x 56 mm, 77 parts, among them J1 Conn_01x05, J10 Conn_01x04, J6 CONN_02X02, J7 USB_B_Micro, J8 Conn_ARM_JTAG_SWD_10, J9 CONN_01X02, P1 Conn_02x20_Odd_Even, Q1 MMDT5401, Q2 FDG1024NZ, Q4 FDG1023NZ, SW1 SW_DIP_x01, U1 CAT24C256, U2 AP131-33, U3 STM32F103CBTx, U4 SN74LVC2T45, U5 SN74LVC2T45, U6 SN74LVC2T45, U7 SN74LVC2T45, U8 USBLC6-2SC6, Y1 8Mhz

Commit message: RPi placed
Parts:
- removed C17, C18, C19: 100n, Capacitor_SMD:C_0603_1608Metric_Pad1.05x0.95mm_HandSolder
- removed MK1, MK2, MK3, MK4: M2.5, MountingHole:MountingHole_2.7mm_M2.5
- removed R12, R13: 22E, Resistor_SMD:R_0603_1608Metric_Pad1.05x0.95mm_HandSolder
- removed R19, R20, R21, R22, R25, R26, R27: 100E, Resistor_SMD:R_0603_1608Metric_Pad1.05x0.95mm_HandSolder
- removed R23, R24: 22, Resistor_SMD:R_0603_1608Metric_Pad1.05x0.95mm_HandSolder
- removed R29: 1K, Resistor_SMD:R_0603_1608Metric_Pad1.05x0.95mm_HandSolder
- removed R6A1, R6B1: 330E, Resistor_SMD:R_0603_1608Metric_Pad1.05x0.95mm_HandSolder
- removed SW1: SW_DIP_x01, Button_Switch_SMD:SW_SPST_FSMSM
- added D5: D, Diode_SMD:D_2114_3652Metric_Pad1.85x3.75mm_HandSolder, F.Cu at (370.4, 152.4)
- added D6: D, Diode_SMD:D_2114_3652Metric_Pad1.85x3.75mm_HandSolder, F.Cu at (355.7, 168.9)
- added F1: Fuse, Fuse:Fuse_1206_3216Metric_Pad1.42x1.75mm_HandSolder, F.Cu at (329.0, 173.6)
- added F2: Fuse, Fuse:Fuse_1206_3216Metric_Pad1.42x1.75mm_HandSolder, F.Cu at (334.3, 173.6)
- added F3: Fuse, Fuse:Fuse_1206_3216Metric_Pad1.42x1.75mm_HandSolder, F.Cu at (339.7, 173.6)
- added H1: MountingHole, MountingHole:MountingHole_2.7mm_M2.5, F.Cu at (203.5, 146.5)
- added H2: MountingHole, MountingHole:MountingHole_2.7mm_M2.5, F.Cu at (261.5, 146.5)
- added H3: MountingHole, MountingHole:MountingHole_2.7mm_M2.5, F.Cu at (203.5, 97.5)
- added H4: MountingHole, MountingHole:MountingHole_2.7mm_M2.5, F.Cu at (261.5, 97.5)
- added J11: SWD-7, Connector_JST:JST_PH_B6B-PH-K_1x06_P2.00mm_Vertical, F.Cu at (448.5, 92.5)
- added J12: SWD-8, Connector_JST:JST_PH_B6B-PH-K_1x06_P2.00mm_Vertical, F.Cu at (433.2, 101.4)
- added J13: Conn_reset, Connector_JST:JST_PH_B2B-PH-K_1x02_P2.00mm_Vertical, F.Cu at (497.8, 110.9)
- added J14: Conn_LEDs, Connector_JST:JST_PH_B4B-PH-K_1x04_P2.00mm_Vertical, F.Cu at (444.7, 148.7)
- added J15: Audio_input, Connector_JST:JST_PH_B2B-PH-K_1x02_P2.00mm_Vertical, F.Cu at (433.7, 180.6)
- added J16: alim_rpi, Connector_Phoenix_MSTB:PhoenixContact_MSTBA_2,5_2-G_1x02_P5.00mm_Horizontal, F.Cu at (330.5, 152.8)
- added J17: alim_audio, Connector_Phoenix_MSTB:PhoenixContact_MSTBA_2,5_2-G_1x02_P5.00mm_Horizontal, F.Cu at (357.4, 152.8)
- added J18: alim_led, Connector_Phoenix_MSTB:PhoenixContact_MSTBA_2,5_2-G_1x02_P5.00mm_Horizontal, F.Cu at (344.0, 152.8)
- added J2: Conn_start, Connector_JST:JST_PH_B2B-PH-K_1x02_P2.00mm_Vertical, F.Cu at (375.4, 101.9)
- added J3: CAN_conn, Connector_JST:JST_XH_B04B-XH-A_1x04_P2.50mm_Vertical, F.Cu at (385.0, 153.1)
- added J4: CAN_conn, Connector_JST:JST_XH_B04B-XH-A_1x04_P2.50mm_Vertical, F.Cu at (385.0, 163.3)
- added J5: SWD-1, Connector_JST:JST_PH_B6B-PH-K_1x06_P2.00mm_Vertical, F.Cu at (433.2, 119.3)
- added JP1: reset_method, Connector_PinHeader_2.54mm:PinHeader_1x03_P2.54mm_Vertical, F.Cu at (349.0, 91.9)
- added JP2: Jumper_RX, Connector_PinHeader_2.54mm:PinHeader_1x02_P2.54mm_Vertical, F.Cu at (490.1, 110.3)
- added JP3: Jumper_TX, Connector_PinHeader_2.54mm:PinHeader_1x02_P2.54mm_Vertical, F.Cu at (485.6, 123.1)
- added JP4: Jumper_SWDIO, Connector_PinHeader_2.54mm:PinHeader_1x02_P2.54mm_Vertical, F.Cu at (491.4, 101.1)
- added JP5: Jumper_SWCLK, Connector_PinHeader_2.54mm:PinHeader_1x02_P2.54mm_Vertical, F.Cu at (479.3, 113.9)
- added JP6: Jumper_NC_Dual, Jumper:SolderJumper-3_P1.3mm_Open_RoundedPad1.0x1.5mm_NumberLabels, F.Cu at (345.5, 167.8)
- added JP7: Jumper_NC_Dual, Jumper:SolderJumper-3_P1.3mm_Open_RoundedPad1.0x1.5mm_NumberLabels, F.Cu at (332.7, 167.8)
- added LS1: Speaker, Connector_JST:JST_PH_B2B-PH-K_1x02_P2.00mm_Vertical, F.Cu at (455.3, 168.1)
- added Q3: NMOS-T252, Package_TO_SOT_SMD:TO-252-2, F.Cu at (459.1, 139.2)
- added Q5: BSS138, Package_TO_SOT_SMD:SOT-23, F.Cu at (398.8, 170.2)
- added U10: SN74LVC1G00, Package_TO_SOT_SMD:SOT-23-5_HandSoldering, F.Cu at (475.9, 123.7)
- added U11: MC34152, Package_SO:SOIC-8_3.9x4.9mm_P1.27mm, F.Cu at (457.4, 149.3)
- added U12: MC34152, Package_SO:SOIC-8_3.9x4.9mm_P1.27mm, F.Cu at (468.8, 138.2)
- added U13: LM4991, Package_SO:SOIC-8_3.9x4.9mm_P1.27mm, F.Cu at (443.2, 181.2)
- added U9: SN74CB3Q3257, Package_SO:TSSOP-16_4.4x5mm_P0.65mm, F.Cu at (479.6, 105.9)
- C1, C10, C3, C5, C6, C7: value 100n -> C; footprint Capacitor_SMD:C_0603_1608Metric_Pad1.05x0.95mm_HandSolder -> Capacitor_SMD:C_0805_2012Metric_Pad1.15x1.40mm_HandSolder; moved to F.Cu
- C11: value 1u -> C; footprint Capacitor_SMD:C_0603_1608Metric_Pad1.05x0.95mm_HandSolder -> Capacitor_SMD:C_0805_2012Metric_Pad1.15x1.40mm_HandSolder; moved to F.Cu
- C12: value 100n -> 10µ; footprint Capacitor_SMD:C_0603_1608Metric_Pad1.05x0.95mm_HandSolder -> Capacitor_SMD:CP_Elec_8x10
- C13: footprint Capacitor_SMD:C_0603_1608Metric_Pad1.05x0.95mm_HandSolder -> Capacitor_SMD:C_0805_2012Metric_Pad1.15x1.40mm_HandSolder
- C14: value 100n -> 0,39u; footprint Capacitor_SMD:C_0603_1608Metric_Pad1.05x0.95mm_HandSolder -> Capacitor_SMD:C_0805_2012Metric_Pad1.15x1.40mm_HandSolder
- C15, C16: value 100n -> 1u; footprint Capacitor_SMD:C_0603_1608Metric_Pad1.05x0.95mm_HandSolder -> Capacitor_SMD:CP_Elec_8x10
- C2, C9: value 4u7 -> C; footprint Capacitor_SMD:C_0603_1608Metric_Pad1.05x0.95mm_HandSolder -> Capacitor_SMD:C_0805_2012Metric_Pad1.15x1.40mm_HandSolder
- C4: value 10n -> C; footprint Capacitor_SMD:C_0603_1608Metric_Pad1.05x0.95mm_HandSolder -> Capacitor_SMD:C_0805_2012Metric_Pad1.15x1.40mm_HandSolder
- C8: value 4u7 -> C; footprint Capacitor_SMD:C_0603_1608Metric_Pad1.05x0.95mm_HandSolder -> Capacitor_SMD:C_0805_2012Metric_Pad1.15x1.40mm_HandSolder; moved to F.Cu
- D1: value Green -> LED; footprint Diode_SMD:D_0603_1608Metric_Pad1.05x0.95mm_HandSolder -> LED_SMD:LED_0805_2012Metric_Pad1.15x1.40mm_HandSolder
- D2: value Red -> D; footprint Diode_SMD:D_0603_1608Metric_Pad1.05x0.95mm_HandSolder -> Diode_SMD:D_2114_3652Metric_Pad1.85x3.75mm_HandSolder
- D3: value Orange -> LED; footprint Diode_SMD:D_0603_1608Metric_Pad1.05x0.95mm_HandSolder -> LED_SMD:LED_0805_2012Metric_Pad1.15x1.40mm_HandSolder
- D4: value Yellow -> LED; footprint Diode_SMD:D_0603_1608Metric_Pad1.05x0.95mm_HandSolder -> LED_SMD:LED_0805_2012Metric_Pad1.15x1.40mm_HandSolder
- J1: value Conn_01x05 -> Conn_sel; footprint Connector_PinHeader_2.54mm:PinHeader_1x05_P2.54mm_Vertical -> Connector_JST:JST_PH_B2B-PH-K_1x02_P2.00mm_Vertical
- J10: value Conn_01x04 -> SWD-6; footprint Connector_Molex:Molex_KK-254_AE-6410-04A_1x04_P2.54mm_Vertical -> Connector_JST:JST_PH_B6B-PH-K_1x06_P2.00mm_Vertical
- J6: value CONN_02X02 -> SWD-2; footprint Connector_PinHeader_2.54mm:PinHeader_2x02_P2.54mm_Vertical -> Connector_JST:JST_PH_B6B-PH-K_1x06_P2.00mm_Vertical
- J7: value USB_B_Micro -> SWD-3; footprint Connector_USB:USB_Micro-B_Molex-105017-0001 -> Connector_JST:JST_PH_B6B-PH-K_1x06_P2.00mm_Vertical
- J8: value Conn_ARM_JTAG_SWD_10 -> SWD-4; footprint Connector_IDC:IDC-Header_2x05_P2.54mm_Vertical -> Connector_JST:JST_PH_B6B-PH-K_1x06_P2.00mm_Vertical
- J9: value CONN_01X02 -> SWD-5; footprint Connector_PinHeader_2.54mm:PinHeader_1x02_P2.54mm_Vertical -> Connector_JST:JST_PH_B6B-PH-K_1x06_P2.00mm_Vertical
- Q1: value MMDT5401 -> NMOS-T252; footprint Package_TO_SOT_SMD:SOT-363_SC-70-6 -> Package_TO_SOT_SMD:TO-252-2
- Q2: value FDG1024NZ -> NMOS-T252; footprint Package_TO_SOT_SMD:SOT-363_SC-70-6 -> Package_TO_SOT_SMD:TO-252-2
- Q4: value FDG1023NZ -> BSS138; footprint Package_TO_SOT_SMD:SOT-363_SC-70-6 -> Package_TO_SOT_SMD:SOT-23
- R1: value 4k7 -> R; footprint Resistor_SMD:R_0603_1608Metric_Pad1.05x0.95mm_HandSolder -> Resistor_SMD:R_0805_2012Metric_Pad1.15x1.40mm_HandSolder; moved to F.Cu
- R10: value 1k5 -> 20k; footprint Resistor_SMD:R_0603_1608Metric_Pad1.05x0.95mm_HandSolder -> Resistor_SMD:R_0805_2012Metric_Pad1.15x1.40mm_HandSolder
- R11: value DNP -> 20k; footprint Resistor_SMD:R_0603_1608Metric_Pad1.05x0.95mm_HandSolder -> Resistor_SMD:R_0805_2012Metric_Pad1.15x1.40mm_HandSolder
- R14: value 4k7 -> R; footprint Resistor_SMD:R_0603_1608Metric_Pad1.05x0.95mm_HandSolder -> Resistor_SMD:R_0805_2012Metric_Pad1.15x1.40mm_HandSolder
- R15, R16, R17, R3: value 10k -> R; footprint Resistor_SMD:R_0603_1608Metric_Pad1.05x0.95mm_HandSolder -> Resistor_SMD:R_0805_2012Metric_Pad1.15x1.40mm_HandSolder
- R18: value 100E -> R; footprint Resistor_SMD:R_0603_1608Metric_Pad1.05x0.95mm_HandSolder -> Resistor_SMD:R_0805_2012Metric_Pad1.15x1.40mm_HandSolder
- R2: value 10k -> R; footprint Resistor_SMD:R_0603_1608Metric_Pad1.05x0.95mm_HandSolder -> Resistor_SMD:R_0805_2012Metric_Pad1.15x1.40mm_HandSolder; moved to F.Cu
- R4, R5: value 330E -> R; footprint Resistor_SMD:R_0603_1608Metric_Pad1.05x0.95mm_HandSolder -> Resistor_SMD:R_0805_2012Metric_Pad1.15x1.40mm_HandSolder
- R6, R8: value 3.9K -> R; footprint Resistor_SMD:R_0603_1608Metric_Pad1.05x0.95mm_HandSolder -> Resistor_SMD:R_0805_2012Metric_Pad1.15x1.40mm_HandSolder
- R7, R9: value DNP -> R; footprint Resistor_SMD:R_0603_1608Metric_Pad1.05x0.95mm_HandSolder -> Resistor_SMD:R_0805_2012Metric_Pad1.15x1.40mm_HandSolder
- U1: value CAT24C256 -> MCP2515-EST; footprint Package_SO:SOIC-8_3.9x4.9mm_P1.27mm -> Package_SO:TSSOP-20_4.4x6.5mm_P0.65mm
- U2: value AP131-33 -> MCP2551-I-SN; footprint Package_TO_SOT_SMD:SOT-23-5 -> Package_SO:SOIC-8_3.9x4.9mm_P1.27mm
- U3: value STM32F103CBTx -> SN74CB3Q3257; footprint Package_QFP:LQFP-48_7x7mm_P0.5mm -> Package_SO:TSSOP-16_4.4x5mm_P0.65mm
- U4, U6: value SN74LVC2T45 -> SN74CB3Q3257; footprint Package_TO_SOT_SMD:SOT-23-8_Handsoldering -> Package_SO:TSSOP-16_4.4x5mm_P0.65mm
- U5, U7: value SN74LVC2T45 -> SN74AC08; footprint Package_TO_SOT_SMD:SOT-23-8_Handsoldering -> Package_SO:SOIC-14_3.9x8.7mm_P1.27mm
- U8: value USBLC6-2SC6 -> SN74CB3Q3257; footprint Package_TO_SOT_SMD:SOT-23-6 -> Package_SO:TSSOP-16_4.4x5mm_P0.65mm
- Y1: value 8Mhz -> Crystal_8MHz; footprint Oscillator:Oscillator_SMD_EuroQuartz_XO32-4Pin_3.2x2.5mm_HandSoldering -> Crystal:Crystal_HC49-U_Vertical
- moved U5 266.5 mm to (480.7, 95.0), turned to 0 degrees
- moved R9 265.6 mm to (474.8, 136.4), turned to 0 degrees
- moved U4 265.5 mm to (490.9, 93.1), turned to 0 degrees
- moved U7 255.6 mm to (465.3, 103.9), turned to 0 degrees
- moved R7 255.3 mm to (452.6, 156.5), turned to 0 degrees
- moved C11 255.3 mm to (466.9, 145.4)
- moved J6 242.8 mm to (448.5, 110.4), turned to 0 degrees
- moved U6 241.9 mm to (464.3, 124.0), turned to 0 degrees
- moved C14 240.0 mm to (462.4, 166.9), turned to 0 degrees
- moved C10 238.3 mm to (448.5, 156.4)
- moved J8 237.8 mm to (448.5, 101.4), turned to 0 degrees
- moved Q1 236.0 mm to (447.5, 139.2), turned to 0 degrees
- moved U3 234.0 mm to (452.0, 120.0)
- moved C7 233.8 mm to (449.2, 127.2), turned to 0 degrees
- moved R11 233.0 mm to (454.7, 175.8), turned to 0 degrees
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Connections:
- C10 pad 2: +3V3 -> +7.5V
- C11 pad 2: +3V3 -> +7.5V
- C12 pad 1: GND -> +5VD
- C12 pad 2: +3V3 -> GND
- C13 pad 1: GND -> +5VD
- C13 pad 2: +3V3 -> GND
- C14 pad 1: GND -> Net-(C14-Pad1)
- C14 pad 2: +3V3 -> Net-(C14-Pad2)
- C15 pad 1: GND -> Net-(C15-Pad1)
- C15 pad 2: +3V3 -> GND
- C16 pad 1: GND -> +5VL
- C16 pad 2: /BlackMagicProbev2.1/xTPWR -> GND
- C2 pad 1: +5V -> Net-(C2-Pad1)
- C3 pad 2: /BlackMagicProbev2.1/~RST -> +3V3
- C4 pad 1: Net-(C4-Pad1) -> GND
- C4 pad 2: GND -> +5V
- C9 pad 1: +3V3 -> GND
- C9 pad 2: GND -> +3V3
- D2 pad 1: GND -> +5V
- D2 pad 2: Net-(D2-Pad2) -> GND
- J1 pad 1: /BlackMagicProbev2.1/SWDIO -> /GPIO6
- J10 pad 1: /BlackMagicProbev2.1/TPWR -> Net-(J10-Pad1)
- J10 pad 2: /BlackMagicProbev2.1/TXD -> GND
- J10 pad 3: /BlackMagicProbev2.1/RXD -> Net-(J10-Pad3)
- J10 pad 4: GND -> Net-(J10-Pad4)
- J6 pad 1: /P3V3 -> Net-(J6-Pad1)
- J6 pad 2: /P3V3_HAT -> GND
- J6 pad 3: +5V -> Net-(J6-Pad3)
- J6 pad 4: /P5V_HAT -> Net-(J6-Pad4)
- J7 pad 1: +5V -> Net-(J7-Pad1)
- J7 pad 2: Net-(J7-Pad2) -> GND
- J7 pad 4: GND -> Net-(J7-Pad4)
- J7 pad 5: GND -> Net-(J7-Pad5)
- J7 pad 6: GND -> Net-(J7-Pad6)
- J8 pad 1: /BlackMagicProbev2.1/TPWR -> Net-(J8-Pad1)
- J8 pad 2: /BlackMagicProbev2.1/TMS -> GND
- J8 pad 3: GND -> Net-(J8-Pad3)
- J8 pad 4: /BlackMagicProbev2.1/TCK -> Net-(J8-Pad4)
- J8 pad 5: GND -> Net-(J8-Pad5)
- J8 pad 6: /BlackMagicProbev2.1/TDO -> Net-(J8-Pad6)
- J9 pad 1: GND -> Net-(J9-Pad1)
- J9 pad 2: Net-(J9-Pad2) -> GND
- P1 pad 1: /P3V3_HAT -> +3V3
- P1 pad 17: /P3V3_HAT -> +3V3
- P1 pad 2: /P5V_HAT -> +5V
- P1 pad 4: /P5V_HAT -> +5V
- Q1 pad 1: +5V -> Net-(Q1-Pad1)
- Q1 pad 2: Net-(Q1-Pad2) -> Net-(J14-Pad2)
- Q1 pad 3: Net-(Q1-Pad3) -> GND
- Q2 pad 1: GND -> Net-(Q2-Pad1)
- Q2 pad 2: /BlackMagicProbev2.1/iRST -> Net-(J14-Pad3)
- Q4 pad 1: Net-(Q4-Pad1) -> +3V3
- Q4 pad 2: /BlackMagicProbev2.1/PWR_BR -> Net-(Q4-Pad2)
- Q4 pad 3: /BlackMagicProbev2.1/TPWR -> Net-(Q4-Pad3)
- R1 pad 1: /BlackMagicProbev2.1/TPWR -> /GPIO6
- R1 pad 2: Net-(C1-Pad1) -> +3V3
- R10 pad 2: Net-(R10-Pad2) -> Net-(C14-Pad1)
- R11 pad 1: Net-(J9-Pad2) -> Net-(LS1-Pad2)
- R11 pad 2: GND -> Net-(R10-Pad1)
- R14 pad 2: /BlackMagicProbev2.1/VBUS -> Net-(D1-Pad2)
- R15 pad 1: /BlackMagicProbev2.1/VBUS -> Net-(D5-Pad1)
- R15 pad 2: GND -> Net-(D3-Pad2)
- R16 pad 1: /BlackMagicProbev2.1/xTPWR -> Net-(D6-Pad1)
- R16 pad 2: /BlackMagicProbev2.1/xRST -> Net-(D4-Pad2)
- R17 pad 1: Net-(Q4-Pad1) -> Net-(Q5-Pad2)
- R17 pad 2: /BlackMagicProbev2.1/PWR_BR -> +3V3
- R18 pad 1: /BlackMagicProbev2.1/TPWR -> +5V
- R18 pad 2: /BlackMagicProbev2.1/xTPWR -> Net-(Q5-Pad3)
- R2 pad 1: Net-(C1-Pad1) -> /GPIO26
- R2 pad 2: GND -> +3V3
- R3 pad 1: +3V3 -> /SWD/GRST
- R3 pad 2: Net-(R3-Pad2) -> +3V3
- R4 pad 1: Net-(D3-Pad2) -> Net-(Q4-Pad2)
- R4 pad 2: /BlackMagicProbev2.1/LED1 -> +3V3
- R5 pad 1: Net-(D4-Pad2) -> +5V
- R5 pad 2: /BlackMagicProbev2.1/LED0 -> Net-(Q4-Pad3)
- R6 pad 1: /P3V3_HAT -> Net-(R6-Pad1)
- R6 pad 2: /ID_SC -> GND
- R7 pad 1: /P3V3_HAT -> GND
- R7 pad 2: /P3V3 -> /GPIO19(SPI1_MISO)
- R8 pad 1: /P3V3_HAT -> /GPIO16
- R8 pad 2: /ID_SD -> GND
- R9 pad 1: /P5V_HAT -> GND
- R9 pad 2: +5V -> /GPIO13(PWM1)
- U1 pad 1: GND -> Net-(Q5-Pad2)
- U1 pad 2: GND -> Net-(Q4-Pad2)
- U1 pad 3: GND -> Net-(U1-Pad3)
- U1 pad 4: GND -> Net-(U1-Pad4)
- U1 pad 5: /ID_SC -> Net-(U1-Pad5)
- U1 pad 6: /ID_SD -> Net-(U1-Pad6)
- U1 pad 7: Net-(J9-Pad2) -> Net-(U1-Pad7)
- U1 pad 8: /P3V3_HAT -> Net-(C1-Pad1)
- U2 pad 1: +5V -> Net-(Q5-Pad3)
- U2 pad 4: Net-(C4-Pad1) -> Net-(Q4-Pad3)
- U2 pad 5: +3V3 -> Net-(U2-Pad5)
- U3 pad 1: +3V3 -> /SWD/~s2
- U3 pad 10: Net-(U3-Pad10) -> Net-(J9-Pad6)
- U3 pad 11: /BlackMagicProbev2.1/iTMS_DIR -> Net-(J10-Pad6)
- U3 pad 12: /BlackMagicProbev2.1/iRST -> Net-(J11-Pad6)
- U3 pad 13: /BlackMagicProbev2.1/iTDI -> Net-(J12-Pad6)
- U3 pad 14: /BlackMagicProbev2.1/iTMS -> /GPIO17(GEN0)
- U3 pad 15: /BlackMagicProbev2.1/iTCK -> /GPIO22(GEN3)
- U3 pad 16: /BlackMagicProbev2.1/iTDO -> +3V3
- U3 pad 2: Net-(U3-Pad2) -> /GPIO27(GEN2)
- U3 pad 3: Net-(U3-Pad3) -> Net-(J8-Pad6)
- U3 pad 4: Net-(U3-Pad4) -> Net-(J7-Pad6)
- U3 pad 5: /BlackMagicProbev2.1/HSE_IN -> Net-(J6-Pad6)
- U3 pad 6: /BlackMagicProbev2.1/HSE_OUT -> Net-(J5-Pad6)
- U3 pad 7: /BlackMagicProbev2.1/~RST -> Net-(JP2-Pad2)
- U3 pad 9: +3V3 -> Net-(JP2-Pad2)
- U4 pad 1: +3V3 -> /SWD/~s2
- U4 pad 2: GND -> /GPIO27(GEN2)
- U4 pad 3: /BlackMagicProbev2.1/iTXD -> Net-(J8-Pad5)
- U4 pad 4: GND -> Net-(J7-Pad5)
- U4 pad 5: +3V3 -> Net-(J6-Pad5)
- U4 pad 6: /BlackMagicProbev2.1/xTXD -> Net-(J5-Pad5)
- U4 pad 7: GND -> Net-(JP3-Pad2)
- U4 pad 8: /BlackMagicProbev2.1/xTPWR -> GND
- U5 pad 1: +3V3 -> Net-(U5-Pad1)
- U5 pad 2: /BlackMagicProbev2.1/iTDI -> /SWD/GRST
- U5 pad 3: /BlackMagicProbev2.1/iTCK -> Net-(J11-Pad4)
- U5 pad 4: GND -> Net-(U5-Pad4)
- U5 pad 5: +3V3 -> /SWD/GRST
- U5 pad 6: /BlackMagicProbev2.1/xTCK -> Net-(J12-Pad4)
- U5 pad 7: /BlackMagicProbev2.1/xTDI -> GND
- U5 pad 8: /BlackMagicProbev2.1/xTPWR -> Net-(J9-Pad4)
- U6 pad 1: +3V3 -> /SWD/~s2
- U6 pad 2: /BlackMagicProbev2.1/iTDO -> /GPIO27(GEN2)
- U6 pad 3: /BlackMagicProbev2.1/iRXD -> Net-(U6-Pad3)
- U6 pad 4: GND -> Net-(U6-Pad4)
- U6 pad 5: GND -> Net-(U6-Pad5)
- U6 pad 6: /BlackMagicProbev2.1/xRXD -> Net-(U6-Pad6)
- U6 pad 7: /BlackMagicProbev2.1/xTDO -> /SWD/nrst
- U6 pad 8: /BlackMagicProbev2.1/xTPWR -> GND
- U7 pad 1: +3V3 -> Net-(U6-Pad6)
- U7 pad 2: GND -> /SWD/GRST
- U7 pad 3: /BlackMagicProbev2.1/iTMS -> Net-(J5-Pad4)
- U7 pad 4: GND -> Net-(U6-Pad5)
- U7 pad 5: /BlackMagicProbev2.1/iTMS_DIR -> /SWD/GRST
- U7 pad 6: /BlackMagicProbev2.1/xTMS -> Net-(J6-Pad4)
- U7 pad 8: /BlackMagicProbev2.1/xTPWR -> Net-(J7-Pad4)
- U8 pad 1: Net-(J7-Pad3) -> /SWD/~s2
- U8 pad 2: GND -> /GPIO27(GEN2)
- U8 pad 3: Net-(J7-Pad2) -> Net-(J8-Pad3)
- U8 pad 4: Net-(R10-Pad1) -> Net-(J7-Pad3)
- U8 pad 5: +5V -> Net-(J6-Pad3)
- Y1 pad 1: /BlackMagicProbev2.1/HSE_OUT -> Net-(C1-Pad1)
- Y1 pad 2: GND -> Net-(C2-Pad1)
Routing:
- net +3V3: track 116.1 -> 0.00 mm, vias 12 -> 0
- net GND: track 99.9 -> 0.00 mm, vias 17 -> 0
- net /BlackMagicProbev2.1/TPWR: track 84.1 -> 0.00 mm, vias 1 -> 0
- net +5V: track 74.8 -> 0.00 mm, vias 2 -> 0
- net /P3V3_HAT: track 38.8 -> 0.00 mm
- net /BlackMagicProbev2.1/VBUS: track 36.1 -> 0.00 mm
- net /BlackMagicProbev2.1/PWR_BR: track 34.7 -> 0.00 mm, vias 2 -> 0
- net /BlackMagicProbev2.1/USB+: track 30.8 -> 0.00 mm
- net Net-(R10-Pad2): track 30.4 -> 0.00 mm
- net /BlackMagicProbev2.1/USB-: track 30.4 -> 0.00 mm
- net /BlackMagicProbev2.1/xTPWR: track 29.4 -> 0.00 mm
- net /BlackMagicProbev2.1/iRST: track 27.0 -> 0.00 mm, vias 2 -> 0
- net /BlackMagicProbev2.1/~RST: track 26.0 -> 0.00 mm, vias 1 -> 0
- net /BlackMagicProbev2.1/LED0: track 24.0 -> 0.00 mm, vias 2 -> 0
- net /BlackMagicProbev2.1/LED1: track 23.1 -> 0.00 mm, vias 2 -> 0
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- removed copper zone on B.Cu, net GND
- removed copper zone on F.Cu, net GND
Other:
- board outline removed

Commit message: placement
Parts:
- removed H1, H2, H3, H4: MountingHole, MountingHole:MountingHole_2.7mm_M2.5
- C10, C11, C13, D2, F1, R7, R8, R9, U11, U12: moved to B.Cu
- moved C14 260.5 mm to (202.0, 175.0), turned to 270 degrees
- moved R11 248.7 mm to (206.0, 175.0), turned to 90 degrees
- moved R10 244.4 mm to (205.0, 171.0), turned to 180 degrees
- moved LS1 243.7 mm to (212.0, 183.0), turned to 180 degrees
- moved J3 239.4 mm to (147.0, 127.1)
- moved J4 239.4 mm to (147.0, 137.3)
- moved U13 232.3 mm to (211.0, 175.0), turned to 270 degrees
- moved J15 231.7 mm to (202.0, 181.0)
- moved C16 228.2 mm to (219.0, 175.0), turned to 90 degrees
- moved C15 225.0 mm to (211.0, 166.0)
- moved R8 203.8 mm to (262.0, 182.0), turned to 180 degrees
- moved C4 203.1 mm to (226.0, 125.0), turned to 90 degrees
- moved R9 203.0 mm to (277.0, 182.0)
- moved R3 198.2 mm to (231.0, 104.0), turned to 180 degrees
- moved R4 196.7 mm to (227.0, 114.0), turned to 180 degrees
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Connections:
- U11 pad 5: Net-(Q2-Pad1) -> Net-(Q1-Pad1)
- U11 pad 7: Net-(Q1-Pad1) -> Net-(Q2-Pad1)

Commit message: holes added
Parts:
- added H1: MountingHole, MountingHole:MountingHole_2.7mm_M2.5, F.Cu at (203.5, 146.5)
- added H2: MountingHole, MountingHole:MountingHole_2.7mm_M2.5, F.Cu at (261.5, 97.5)
- added H3: MountingHole, MountingHole:MountingHole_2.7mm_M2.5, F.Cu at (261.5, 146.5)
- added H4: MountingHole, MountingHole:MountingHole_2.7mm_M2.5, F.Cu at (203.5, 97.5)
Changed lines of the file:
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@@
     (tracks 0)
     (zones 0)
-    (modules 87)
+    (modules 91)
     (nets 133)
   )
@@
     (uvia_drill 0.1)
   )
+  (module MountingHole:MountingHole_2.7mm_M2.5 (layer F.Cu)
+    (at 261.5 146.5)
+    (descr "Mounting Hole 2.7mm, no annular, M2.5")
+    (tags "mounting hole 2.7mm no annular m2.5")
+    (attr virtual)
+    (fp_text reference H3 (at 0 -3.7) (layer F.SilkS)
+      (effects (font (size 1 1) (thickness 0.15)))
+    )
+    (fp_text value MountingHole (at 0 3.7) (layer F.Fab)
+      (effects (font (size 1 1) (thickness 0.15)))
+    )
+    (fp_circle (center 0 0) (end 2.95 0) (layer F.CrtYd) (width 0.05))
+    (fp_circle (center 0 0) (end 2.7 0) (layer Cmts.User) (width 0.15))
+    (fp_text user %R (at 0.3 0) (layer F.Fab)
+      (effects (font (size 1 1) (thickness 0.15)))
+    )
+    (pad 1 np_thru_hole circle (at 0 0) (size 2.7 2.7) (drill 2.7) (layers *.Cu *.Mask))
+  )
+  (module MountingHole:MountingHole_2.7mm_M2.5 (layer F.Cu)
+    (at 261.5 97.5)
+    (descr "Mounting Hole 2.7mm, no annular, M2.5")
+    (tags "mounting hole 2.7mm no annular m2.5")
+    (attr virtual)
+    (fp_text reference H2 (at 0 -3.7) (layer F.SilkS)
+      (effects (font (size 1 1) (thickness 0.15)))
+    )
+    (fp_text value MountingHole (at 0 3.7) (layer F.Fab)
+      (effects (font (size 1 1) (thickness 0.15)))
+    )
+    (fp_text user %R (at 0.3 0) (layer F.Fab)
+      (effects (font (size 1 1) (thickness 0.15)))
+    )
+    (fp_circle (center 0 0) (end 2.7 0) (layer Cmts.User) (width 0.15))
+    (fp_circle (center 0 0) (end 2.95 0) (layer F.CrtYd) (width 0.05))
+    (pad 1 np_thru_hole circle (at 0 0) (size 2.7 2.7) (drill 2.7) (layers *.Cu *.Mask))
+  )
+  (module MountingHole:MountingHole_2.7mm_M2.5 (layer F.Cu)
+    (at 203.5 146.5)
+    (descr "Mounting Hole 2.7mm, no annular, M2.5")
+    (tags "mounting hole 2.7mm no annular m2.5")
+    (attr virtual)
+    (fp_text reference H1 (at 0 -3.7) (layer F.SilkS)
+      (effects (font (size 1 1) (thickness 0.15)))
+    )
+    (fp_text value MountingHole (at 0 3.7) (layer F.Fab)
+      (effects (font (size 1 1) (thickness 0.15)))
+    )
+    (fp_circle (center 0 0) (end 2.95 0) (layer F.CrtYd) (width 0.05))
+    (fp_circle (center 0 0) (end 2.7 0) (layer Cmts.User) (width 0.15))
+    (fp_text user %R (at 0.3 0) (layer F.Fab)
+      (effects (font (size 1 1) (thickness 0.15)))
+    )
+    (pad 1 np_thru_hole circle (at 0 0) (size 2.7 2.7) (drill 2.7) (layers *.Cu *.Mask))
+  )
+  (module MountingHole:MountingHole_2.7mm_M2.5 (layer F.Cu)
+    (at 203.5 97.5)
+    (descr "Mounting Hole 2.7mm, no annular, M2.5")
+    (tags "mounting hole 2.7mm no annular m2.5")
+    (attr virtual)
+    (fp_text reference H4 (at 0 -3.7) (layer F.SilkS)
+      (effects (font (size 1 1) (thickness 0.15)))
+    )
+    (fp_text value MountingHole (at 0 3.7) (layer F.Fab)
+      (effects (font (size 1 1) (thickness 0.15)))
+    )
+    (fp_text user %R (at 0.3 0) (layer F.Fab)
+      (effects (font (size 1 1) (thickness 0.15)))
+    )
+    (fp_circle (center 0 0) (end 2.7 0) (layer Cmts.User) (width 0.15))
+    (fp_circle (center 0 0) (end 2.95 0) (layer F.CrtYd) (width 0.05))
+    (pad 1 np_thru_hole circle (at 0 0) (size 2.7 2.7) (drill 2.7) (layers *.Cu *.Mask))
+  )
   (module Capacitor_SMD:CP_Elec_8x10 (layer F.Cu)

Commit message: route longer than expected
Parts:
- moved JP2 361.1 mm to (129.2, 124.4)
- moved J13 355.0 mm to (142.8, 103.7)
- moved JP3 354.8 mm to (130.9, 111.7)
- moved JP4 354.8 mm to (136.7, 89.6)
- moved JP5 354.8 mm to (124.6, 102.4)
- moved JP1 354.8 mm to (141.3, 110.5)
- moved U4 301.3 mm to (190.5, 116.8), turned to 270 degrees
- moved J7 297.2 mm to (168.0, 120.0), turned to 90 degrees
- moved U5 296.9 mm to (194.5, 174.0), turned to 180 degrees
- moved U9 294.3 mm to (190.8, 162.5), turned to 270 degrees
- moved U10 293.1 mm to (185.3, 162.1), turned to 90 degrees
- moved J6 281.8 mm to (168.0, 136.5), turned to 90 degrees
- moved J8 280.6 mm to (168.0, 104.0), turned to 90 degrees
- moved U8 278.3 mm to (190.8, 145.2), turned to 270 degrees
- moved J11 278.1 mm to (187.0, 187.0), turned to 180 degrees
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Connections:
- U7 pad 1: Net-(U6-Pad6) -> Net-(U6-Pad5)
- U7 pad 11: Net-(J8-Pad4) -> Net-(J7-Pad4)
- U7 pad 12: Net-(U6-Pad3) -> Net-(U6-Pad4)
- U7 pad 3: Net-(J5-Pad4) -> Net-(J6-Pad4)
- U7 pad 4: Net-(U6-Pad5) -> Net-(U6-Pad6)
- U7 pad 6: Net-(J6-Pad4) -> Net-(J5-Pad4)
- U7 pad 8: Net-(J7-Pad4) -> Net-(J8-Pad4)
- U7 pad 9: Net-(U6-Pad4) -> Net-(U6-Pad3)
Routing:
- net Net-(J12-Pad6): track 0.00 -> 108.7 mm, vias 0 -> 3
- net /GPIO22(GEN3): track 0.00 -> 102.2 mm, vias 0 -> 8
- net /SWD/~s2: track 0.00 -> 95.4 mm, vias 0 -> 6
- net Net-(J11-Pad6): track 0.00 -> 95.0 mm, vias 0 -> 1
- net /GPIO17(GEN0): track 0.00 -> 94.4 mm, vias 0 -> 8
- net /GPIO27(GEN2): track 0.00 -> 91.3 mm, vias 0 -> 6
- net Net-(J12-Pad5): track 0.00 -> 90.1 mm, vias 0 -> 3
- net Net-(J10-Pad6): track 0.00 -> 88.8 mm, vias 0 -> 1
- net Net-(J10-Pad5): track 0.00 -> 78.1 mm, vias 0 -> 2
- net Net-(J8-Pad1): track 0.00 -> 76.5 mm, vias 0 -> 2
- net Net-(J11-Pad5): track 0.00 -> 76.3 mm, vias 0 -> 1
- net Net-(J9-Pad6): track 0.00 -> 71.6 mm, vias 0 -> 1
- net Net-(J5-Pad6): track 0.00 -> 65.7 mm, vias 0 -> 1
- net Net-(J8-Pad3): track 0.00 -> 64.8 mm, vias 0 -> 2
- net Net-(J9-Pad5): track 0.00 -> 61.1 mm, vias 0 -> 2
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Other:
- board text removed: "DISPLAY"
