File: SWD/fezzesarecool-elec.kicad_pcb (KiCad board)
At the start: 2 copper layers, 25 x 100 mm, 23 parts, among them J1 Conn_01x10, J2 Conn_Debug, J3 Conn_Debug, J4 Conn_Debug, J5 Conn_Debug, J6 Conn_Debug, J7 Conn_Debug, J8 Conn_Debug, J9 Conn_Debug, U10 SN74LVC1G00, U3 SN74CB3Q3257, U4 SN74CB3Q3257, U8 SN74CB3Q3257, U9 SN74CB3Q3257

Commit message: fix phenix phoenix, add silk
Parts:
- removed REF**: KiCad-Logo2_8mm_SilkScreen, Symbol:KiCad-Logo2_8mm_SilkScreen
- removed REF**: OSHW-Logo2_9.8x8mm_SilkScreen, Symbol:OSHW-Logo2_9.8x8mm_SilkScreen
- removed REF**: Logo_8,5mm, PhoenixRobotik:Logo_8,5mm
- added LOGO1: Logo_Open_Hardware_Small, PhenixRobotik:Logo_12,7mm, F.Cu at (110.6, 142.8)
- added LOGO2: Logo_Open_Hardware_Small, Symbol:OSHW-Logo_7.5x8mm_SilkScreen, F.Cu at (110.2, 175.8)
- added LOGO3: Logo_Open_Hardware_Small, Symbol:KiCad-Logo2_8mm_SilkScreen, B.Cu at (114.0, 190.2)
- moved C6 65.6 mm to (120.0, 186.1)
- moved C8 65.6 mm to (120.4, 152.0)
- moved C9 65.6 mm to (120.0, 169.2)
- moved C5 65.6 mm to (122.6, 135.0)
- moved H1 65.6 mm to (116.5, 175.5)
- moved H2 65.6 mm to (115.0, 125.8)
- moved J1 65.6 mm to (122.0, 109.5)
- moved J2 65.6 mm to (103.0, 147.8)
- moved J3 65.6 mm to (103.0, 132.0)
- moved J4 65.6 mm to (103.0, 196.0)
- moved J5 65.6 mm to (112.0, 103.0)
- moved J6 65.6 mm to (103.0, 164.0)
- moved J7 65.6 mm to (122.0, 197.0)
- moved J8 65.6 mm to (103.0, 179.8)
- moved J9 65.6 mm to (103.0, 116.0)
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Other:
- outline, holes or cut-outs redrawn
